File: Lutje v1.kicad_sch (KiCad schematic)
At the start: 58 parts, among them J1 Conn_01x02, J2 Conn_Coaxial, J3 Conn_01x02, J4 Conn_01x02, J5 Conn_01x02, J6 Conn_01x03, J8 Conn_01x03, Q1 AON7403, SW1 SW_Push, U1 SX1280, U11 DRV8212DRL, U2 2450FM07D0034, U3 ESP32-U4WDH, U7 DRV8212DRL, U8 AMS1117-3.3, Y1 XC21M4-52.000-F10NNHPL, Y2 40Mhz

Commit message: LDO capacitor resistor. antenna placeholder
Parts:
- added R11: R, Capacitor_SMD:C_0402_1005Metric, symbol Device:R
- AE2: footprint (none) -> RF_Antenna:Texas_SWRA117D_2.4GHz_Left
Connections:
- net +3V3: now also R11.2; no longer C7.1
- net GND: no longer AE1.1 (FEED)
- new net: C7.1, R11.1
- no-connect marks 9 -> 10
Other:
- note added: "pcb MIFA placeholder"
- moved on the sheet: C7, D1, R7
